Commit message: Update (include json library)

File: catkin_ws/src/cpush_config/models/IRB120/irb_120.urdf (robot description, URDF)
Before this commit: robot irb_120, 9 links, 8 joints
Links:
- link base_link: geometry collision mesh filename=package://cpush_config/models/IRB120/meshes/collision/base_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 scale=0.0254 0.0254 0.0254; visual mesh filename=package://cpush_config/models/IRB120/meshes/visual/base_lin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 scale=0.0254 0.0254 0.0254
- link link_1: geometry collision mesh filename=package://cpush_config/models/IRB120/meshes/collision/link_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 scale=0.0254 0.0254 0.0254; visual mesh filename=package://cpush_config/models/IRB120/meshes/visual/link_1.s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 scale=0.0254 0.0254 0.0254
- link link_2: geometry collision mesh filename=package://cpush_config/models/IRB120/meshes/collision/link_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 scale=0.0254 0.0254 0.0254; visual mesh filename=package://cpush_config/models/IRB120/meshes/visual/link_2.s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 scale=0.0254 0.0254 0.0254
- link link_3: geometry collision mesh filename=package://cpush_config/models/IRB120/meshes/collision/link_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 scale=0.0254 0.0254 0.0254; visual mesh filename=package://cpush_config/models/IRB120/meshes/visual/link_3.s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 scale=0.0254 0.0254 0.0254
- link link_4: geometry collision mesh filename=package://cpush_config/models/IRB120/meshes/collision/link_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 scale=0.0254 0.0254 0.0254; visual mesh filename=package://cpush_config/models/IRB120/meshes/visual/link_4.s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 scale=0.0254 0.0254 0.0254
- link link_5: geometry collision mesh filename=package://cpush_config/models/IRB120/meshes/collision/link_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 scale=0.0254 0.0254 0.0254; visual mesh filename=package://cpush_config/models/IRB120/meshes/visual/link_5.s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 scale=0.0254 0.0254 0.0254
- link link_6: geometry collision mesh filename=package://cpush_config/models/IRB120/meshes/collision/link_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 scale=0.0254 0.0254 0.0254; visual mesh filename=package://cpush_config/models/IRB120/meshes/visual/link_6.s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 scale=0.0254 0.0254 0.0254
